Commit message: Add files via upload

File: water_description/urdf/water_all.xacro (robot description, xacro)
@@ -160,5 +160,5 @@
     <inertial>
       <mass value="0.01" />
-      <origin xyz="0 0 0" />
+      <origin xyz="0 0 -0.3" />
       <inertia ixx="0.001" ixy="0.0" ixz="0.0"
                 iyy="0.001" iyz="0.0"
@@ -181,5 +181,5 @@
     <inertial>
       <mass value="0.01" />
-      <origin xyz="0 0 0" />
+      <origin xyz="0 0 -0.3" />
       <inertia ixx="0.001" ixy="0.0" ixz="0.0"
                 iyy="0.001" iyz="0.0"
@@ -202,5 +202,5 @@
     <inertial>
       <mass value="0.01" />
-      <origin xyz="0 0 0" />
+      <origin xyz="0 0 -0.3" />
       <inertia ixx="0.001" ixy="0.0" ixz="0.0"
                 iyy="0.001" iyz="0.0"
@@ -215,15 +215,15 @@
   </link>
   <joint name="holder1_joint" type="fixed">
-    <origin xyz="0.0 0.10 0.62" rpy="0 0 0"/>
+    <origin xyz="0.0 0.01 0.645" rpy="0 0 0"/>
     <parent link="base_link"/>
     <child link="holder1"/>
   </joint>
   <joint name="holder2_joint" type="fixed">
-    <origin xyz="0.08 0.2 0.62" rpy="0 0 0"/>
+    <origin xyz="0.1175 0.2 0.645" rpy="0 0 0"/>
     <parent link="base_link"/>
     <child link="holder2"/>
   </joint>
   <joint name="holder3_joint" type="fixed">
-    <origin xyz="-0.08 0.2 0.62" rpy="0 0 0"/>
+    <origin xyz="-0.1175 0.2 0.645" rpy="0 0 0"/>
     <parent link="base_link"/>
     <child link="holder3"/>
@@ -232,18 +232,18 @@
     <collision>
       <geometry>
-        <box size=".25 .2 .01"/>
-      </geometry>
-      <origin rpy="0 0 0" xyz="0 0 0"/>
-    </collision>
-    <inertial>
-      <mass value="0.01" />
-      <origin xyz="0 0 0" />
-      <inertia ixx="0.001" ixy="0.0" ixz="0.0"
-                iyy="0.001" iyz="0.0"
-                izz="0.001" />
-    </inertial>
-    <visual>
-      <geometry>
-        <box size=".25 .2 .01"/>
+        <box size=".3 .25 .01"/>
+      </geometry>
+      <origin rpy="0 0 0" xyz="0 0 0"/>
+    </collision>
+    <inertial>
+      <mass value="0.01" />
+      <origin xyz="0 0 0" />
+      <inertia ixx="0.001" ixy="0.0" ixz="0.0"
+                iyy="0.001" iyz="0.0"
+                izz="0.001" />
+    </inertial>
+    <visual>
+      <geometry>
+        <box size=".3 .25 .01"/>
       </geometry>
       <origin xyz="0 0 0" rpy="0 0 0"/>
@@ -253,18 +253,18 @@
     <collision>
       <geometry>
-        <box size=".25 .2 .01"/>
-      </geometry>
-      <origin rpy="0 0 0" xyz="0 0 0"/>
-    </collision>
-    <inertial>
-      <mass value="0.01" />
-      <origin xyz="0 0 0" />
-      <inertia ixx="0.001" ixy="0.0" ixz="0.0"
-                iyy="0.001" iyz="0.0"
-                izz="0.001" />
-    </inertial>
-    <visual>
-      <geometry>
-        <box size=".25 .2 .01"/>
+        <box size=".3 .25 .01"/>
+      </geometry>
+      <origin rpy="0 0 0" xyz="0 0 0"/>
+    </collision>
+    <inertial>
+      <mass value="0.01" />
+      <origin xyz="0 0 0" />
+      <inertia ixx="0.001" ixy="0.0" ixz="0.0"
+                iyy="0.001" iyz="0.0"
+                izz="0.001" />
+    </inertial>
+    <visual>
+      <geometry>
+        <box size=".3 .25 .01"/>
       </geometry>
       <origin xyz="0 0 0" rpy="0 0 0"/>
@@ -272,5 +272,5 @@
   </link>
   <joint name="pan1_joint" type="fixed">
-    <origin xyz="0 0.07 0.4" rpy="0 0 0"/>
+    <origin xyz="0 0.1 0.4" rpy="0 0 0"/>
     <parent link="holder1"/>
     <child link="pan1"/>
@@ -317,5 +317,5 @@
   </xacro:realsense_d435>
   <xacro:realsense_d435 sensor_name="d435_high" parent_link="pan2" rate="10">
-    <origin rpy="0 0 ${M_PI/2}" xyz="0 0.1 0.008"/>
+    <origin rpy="0 0 ${M_PI/2}" xyz="0 0.12 0.008"/>
   </xacro:realsense_d435>
   <gazebo reference="wheel_left_link">
